File: Hardware/WifiSensor.kicad_pcb (KiCad board)
At the start: 2 copper layers, 32 x 32 mm, 17 parts, among them J1 Power, J8 Tx Rx GND, SW1 Reset, U1 BME280, U2 LD1117S33TR_SOT223, U4 ESP-12E

Commit message: Rev. B
Parts:
- U2: value LD1117S33TR_SOT223 -> LT1129-3.3_SOT223
- moved U2 0.10 mm to (76.0, 78.4)
Connections:
- U2 pad 1: GNDD -> +BATT
- U2 pad 2: +3V3 -> GNDD
- U2 pad 3: +BATT -> +3V3
Routing:
- net +3V3: track 74.9 -> 78.0 mm, vias 3 -> 2
- net +BATT: track 13.6 -> 11.5 mm, vias 0 -> 2
- net GNDD: track 8.49 -> 8.55 mm, vias 17 -> 16
Other:
- board text added: "GND"
- board text added: "Program"
- board text added: "Reset"
- board text added: "Rx"
- board text added: "Tx"
- board text added: "WiFi Sensor Rev. B Paweł Warzecha"
- board text removed: "WiFi Sensor Rev. A Paweł Warzecha"

Commit message: Revision C
Parts:
- added JP2: DeepSleepEnable, Jumper:SolderJumper-2_P1.3mm_Open_RoundedPad1.0x1.5mm, F.Cu at (54.0, 66.0)
Routing:
- net Net-(JP2-Pad2): track 12.1 -> 21.6 mm
- net Net-(JP2-Pad1): track 0.00 -> 5.23 mm
Other:
- board text added: "DeepSleep Enable"
- board text added: "WiFi Sensor Rev. C Paweł Warzecha"
- board text removed: "WiFi Sensor Rev. B Paweł Warzecha"
