File: Hardware/WifiSensor.sch (KiCad schematic (older format))
At the start: 17 parts, among them J1 Power, J8 Tx Rx GND, SW1 Reset, U1 BME280, U2 LD1117S33TR_SOT223, U4 ESP-12E

Commit message: Rev. B
Parts:
- removed U2: LD1117S33TR_SOT223, Package_TO_SOT_SMD:SOT-223-3_TabPin2, symbol Regulator_Linear:LD1117S33TR_SOT223
- added U2: LT1129-3.3_SOT223, Package_TO_SOT_SMD:SOT-223-3_TabPin2, symbol Regulator_Linear:LT1129-3.3_SOT223
Connections:
- net +3V3: now also U2.3 (VO)
- net +BATT: now also U2.1 (VI)
- net GNDD: now also U2.2 (GND)
Changed lines of the file:
@@
 Sheet 1 1
 Title "Wifi Sensor"
-Date "2022-08-02"
-Rev "Rev. A"
+Date "2022-08-03"
+Rev "Rev. B"
 Comp "Pawel Warzecha"
 Comment1 ""
@@
 	4350 3050 4450 3050
 $Comp
-L Regulator_Linear:LD1117S33TR_SOT223 U2
-U 1 1 62E84AC9
-P 2300 1000
-F 0 "U2" H 2300 1242 50  0000 C CNN
-F 1 "LD1117S33TR_SOT223" H 2300 1151 50  0000 C CNN
-F 2 "Package_TO_SOT_SMD:SOT-223-3_TabPin2" H 2300 1200 50  0001 C CNN
-F 3 "http://www.st.com/st-web-ui/static/active/en/resource/technical/document/datasheet/CD00000544.pdf" H 2400 750 50  0001 C CNN
-	1    2300 1000
-	1    0    0    -1
-$EndComp
-$Comp
 L Connector_Generic:Conn_01x04 J1
 U 1 1 62E863A8
@@
 	1    0    0    -1
 $EndComp
+$Comp
+L Regulator_Linear:LT1129-3.3_SOT223 U2
+U 1 1 62F9462A
+P 2300 1000
+F 0 "U2" H 2300 1242 50  0000 C CNN
+F 1 "LT1129-3.3_SOT223" H 2300 1151 50  0000 C CNN
+F 2 "Package_TO_SOT_SMD:SOT-223-3_TabPin2" H 2300 1225 50  0001 C CIN
+F 3 "https://www.analog.com/media/en/technical-documentation/data-sheets/112935ff.pdf" H 2300 950 50  0001 C CNN
+	1    2300 1000
+	1    0    0    -1
+$EndComp

Commit message: Revision C
Parts:
- added JP2: DeepSleepEnable, Jumper:SolderJumper-2_P1.3mm_Open_RoundedPad1.0x1.5mm, symbol Connector_Generic:Conn_01x02
Connections:
- net at R3.2, SW1.2 (Pin_2), U4.1 (REST): now also JP2.2 (Pin_2)
- net at U4.4 (GPIO16): now also JP2.1 (Pin_1)
Changed lines of the file:
@@
 Sheet 1 1
 Title "Wifi Sensor"
-Date "2022-08-03"
-Rev "Rev. B"
+Date "2022-08-14"
+Rev "Rev. C"
 Comp "Pawel Warzecha"
 Comment1 ""
@@
 Wire Notes Line
 	5050 1850 650  1850
-Text GLabel 1500 3050 0    50   Input ~ 0
+Text GLabel 1850 3050 0    50   Input ~ 0
 SCL
-Text GLabel 1500 3150 0    50   Input ~ 0
+Text GLabel 1850 3150 0    50   Input ~ 0
 SDA
 Wire Wire Line
@@
 	0    -1   -1   0
 $EndComp
-Text Label 1500 3050 0    50   ~ 0
+Text Label 1850 3050 0    50   ~ 0
 SCL
-Text Label 1500 3150 0    50   ~ 0
+Text Label 1850 3150 0    50   ~ 0
 SDA
 Text Notes 650  4000 0    50   ~ 0
@@
 	1700 3400 1700 3450
 Wire Wire Line
-	1500 3150 1900 3150
-Wire Wire Line
-	1500 3050 1900 3050
+	1850 3150 1900 3150
+Wire Wire Line
+	1850 3050 1900 3050
 Wire Wire Line
 	1700 2750 1900 2750
@@
 $EndComp
 Wire Wire Line
-	1450 2550 1900 2550
+	1450 2550 1550 2550
 Wire Wire Line
 	1450 2550 1300 2550
@@
 	1    0    0    -1
 $EndComp
+$Comp
+L Connector_Generic:Conn_01x02 JP2
+U 1 1 62F97B0A
+P 1100 3200
+F 0 "JP2" H 1100 3464 50  0000 C CNN
+F 1 "DeepSleepEnable" H 1100 3373 50  0000 C CNN
+F 2 "Jumper:SolderJumper-2_P1.3mm_Open_RoundedPad1.0x1.5mm" H 1100 3200 50  0001 C CNN
+F 3 "" H 1100 3200 50  0000 C CNN
+	1    1100 3200
+	-1   0    0    1
+$EndComp
+Wire Wire Line
+	1300 3200 1600 3200
+Wire Wire Line
+	1900 2850 1600 2850
+Wire Wire Line
+	1600 2850 1600 3200
+Wire Wire Line
+	1300 3100 1550 3100
+Wire Wire Line
+	1550 3100 1550 2550
+Connection ~ 1550 2550
+Wire Wire Line
+	1550 2550 1900 2550
 $EndSCHEMATC
